File: SAP-U_Project/No_Connects.kicad_sch (KiCad schematic)
At the start: 3 parts, among them U1 74LS08, U5 74LS32, U6 74LS04

Commit message: Checkpoint: Linked footprints to schematics
Parts:
- U1: footprint (none) -> MyFootPrints:SN74LS08N
- U5: footprint (none) -> MyFootPrints:SN74LS32N
- U6: footprint (none) -> MyFootPrints:SN74LS04N
Changed lines of the file:
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@@
 			)
 		)
-		(property "Footprint" ""
+		(property "Footprint" "MyFootPrints:SN74LS08N"
 			(at 29.21 30.48 0)
 			(effects
@@
 			)
 		)
-		(property "Footprint" ""
+		(property "Footprint" "MyFootPrints:SN74LS04N"
 			(at 80.01 45.72 0)
 			(effects
@@
 			)
 		)
-		(property "Footprint" ""
+		(property "Footprint" "MyFootPrints:SN74LS32N"
 			(at 52.07 30.48 0)
 			(effects
@@
 			)
 		)
-		(property "Footprint" ""
+		(property "Footprint" "MyFootPrints:SN74LS04N"
 			(at 78.74 30.48 0)
 			(effects
@@
 			)
 		)
-		(property "Footprint" ""
+		(property "Footprint" "MyFootPrints:SN74LS04N"
 			(at 80.01 62.23 0)
 			(effects
@@
 			)
 		)
-		(property "Footprint" ""
+		(property "Footprint" "MyFootPrints:SN74LS32N"
 			(at 52.07 45.72 0)
 			(effects
@@
 			)
 		)
-		(property "Footprint" ""
+		(property "Footprint" "MyFootPrints:SN74LS32N"
 			(at 52.07 62.23 0)
 			(effects
