File: Arithmetic_Logic_Unit/Register_sch.kicad_sch (KiCad schematic)
At the start: 22 parts, among them U12 74LS245, U13 74LS173, U14 74LS173

Commit message: updated Arithemetic Logic Unit
Parts:
- removed C12, C13, C14: .01µF, Capacitor_THT:C_Disc_D5.0mm_W2.5mm_P2.50mm, symbol Device:C
- removed D17, D18, D19, D20, D21, D22, D23, D24: LED, LED_THT:LED_D5.0mm, symbol Device:LED
- removed R17, R18, R19, R20, R21, R22, R23, R24: 220, Resistor_THT:R_Axial_DIN0207_L6.3mm_D2.5mm_P5.08mm_Vertical, symbol Device:R
- removed U12: 74LS245, Package_DIP:DIP-20_W7.62mm, symbol 74xx:74LS245
- removed U13, U14: 74LS173, Package_DIP:DIP-16_W7.62mm, symbol 74xx:74LS173
Other:
- note removed: "Flip Flop"
- note removed: "Input data from the bus"
- note removed: "Tristate Buffer"
- note removed: "Upper Bytes"
- note removed: "output enable controlled with tristate buffer"
- company: Arsenal Gear -> (none)
- title: Registers -> (none)
